File: NixiePowerSupply.kicad_sch (KiCad schematic)
At the start: 16 parts, among them J1 Conn_01x02, J2 Conn_01x02, Q1 IRF740, Q2 PNP, U1 MC34063AP

Commit message: add Library.pretty
Parts:
- C2, C3: footprint (none) -> Capacitor_SMD:C_0805_2012Metric_Pad1.18x1.45mm_HandSolder
- J1, J2: footprint (none) -> Library:DG301-5.0-2P-1X
- R1, R2: footprint (none) -> Resistor_SMD:R_0805_2012Metric_Pad1.20x1.40mm_HandSolder
- R3, R4: footprint (none) -> Resistor_THT:R_Axial_DIN0207_L6.3mm_D2.5mm_P7.62mm_Horizontal
Changed lines of the file:
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@@
       (effects (font (size 1.27 1.27)) (justify left) hide)
     )
-    (property "Footprint" "" (at 124.1552 151.13 0)
+    (property "Footprint" "Capacitor_SMD:C_0805_2012Metric_Pad1.18x1.45mm_HandSolder" (at 124.1552 151.13 0)
       (effects (font (size 1.27 1.27)) hide)
     )
@@
       (effects (font (size 1.27 1.27)) (justify left) hide)
     )
-    (property "Footprint" "" (at 144.78 125.73 0)
+    (property "Footprint" "Library:DG301-5.0-2P-1X" (at 144.78 125.73 0)
       (effects (font (size 1.27 1.27)) hide)
     )
@@
       (effects (font (size 1.27 1.27)) (justify left) hide)
     )
-    (property "Footprint" "" (at 71.12 123.19 0)
+    (property "Footprint" "Library:DG301-5.0-2P-1X" (at 71.12 123.19 0)
       (effects (font (size 1.27 1.27)) hide)
     )
@@
       (effects (font (size 1.27 1.27)) (justify left) hide)
     )
-    (property "Footprint" "" (at 127.762 147.32 90)
+    (property "Footprint" "Resistor_THT:R_Axial_DIN0207_L6.3mm_D2.5mm_P7.62mm_Horizontal" (at 127.762 147.32 90)
       (effects (font (size 1.27 1.27)) hide)
     )
@@
       (effects (font (size 1.27 1.27)) (justify left) hide)
     )
-    (property "Footprint" "" (at 79.7052 140.97 0)
+    (property "Footprint" "Capacitor_SMD:C_0805_2012Metric_Pad1.18x1.45mm_HandSolder" (at 79.7052 140.97 0)
       (effects (font (size 1.27 1.27)) hide)
     )
@@
       (effects (font (size 1.27 1.27)) (justify left) hide)
     )
-    (property "Footprint" "" (at 102.362 142.24 90)
+    (property "Footprint" "Resistor_SMD:R_0805_2012Metric_Pad1.20x1.40mm_HandSolder" (at 102.362 142.24 90)
       (effects (font (size 1.27 1.27)) hide)
     )
@@
       (effects (font (size 1.27 1.27)) hide)
     )
-    (property "Footprint" "" (at 91.44 117.348 90)
+    (property "Footprint" "Resistor_SMD:R_0805_2012Metric_Pad1.20x1.40mm_HandSolder" (at 91.44 117.348 90)
       (effects (font (size 1.27 1.27)) hide)
     )
@@
       (effects (font (size 1.27 1.27)) (justify left) hide)
     )
-    (property "Footprint" "" (at 127.762 139.7 90)
-      (effects (font (size 1.27 1.27)) hide)
-    )
+    (property "Footprint" "Resistor_THT:R_Axial_DIN0207_L6.3mm_D2.5mm_P7.62mm_Horizontal" (at 127.762 139.7 90)
+      (effects (font (size 1.27 1.27)) hide)
+    )

Commit message: add footprints
Parts:
- removed Q2: PNP, symbol Simulation_SPICE:PNP
- added Q2: 2N3905, Package_TO_SOT_THT:TO-92_Inline, symbol Transistor_BJT:2N3905
- C1, C4: footprint (none) -> Capacitor_THT:CP_Radial_D6.3mm_P2.50mm
- D1: footprint (none) -> Diode_THT:D_DO-41_SOD81_P7.62mm_Horizontal
- D2: footprint (none) -> Diode_THT:D_DO-35_SOD27_P7.62mm_Horizontal
- L1: footprint (none) -> Inductor_SMD:L_12x12mm_H8mm
Connections:
- net GND: now also Q2.3 (C)
- net at D2.2 (A), R2.1, U1.2 (SwE): now also Q2.2 (B)
- net at D2.1 (K), Q1.1 (G): now also Q2.1 (E)
Changed lines of the file:
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@@
   (junction (at 121.92 125.73) (diameter 0) (color 0 0 0 0)
   )
+  (junction (at 104.14 123.19) (diameter 0) (color 0 0 0 0)
+  )
+  (junction (at 129.54 143.51) (diameter 0) (color 0 0 0 0)
+  )
+  (junction (at 104.14 138.43) (diameter 0) (color 0 0 0 0)
+  )
+  (junction (at 104.14 133.35) (diameter 0) (color 0 0 0 0)
+  )
+  (junction (at 134.62 125.73) (diameter 0) (color 0 0 0 0)
+  )
+  (junction (at 78.74 123.19) (diameter 0) (color 0 0 0 0)
+  )
   (junction (at 114.3 133.35) (diameter 0) (color 0 0 0 0)
-  )
-  (junction (at 104.14 123.19) (diameter 0) (color 0 0 0 0)
-  )
-  (junction (at 129.54 143.51) (diameter 0) (color 0 0 0 0)
-  )
-  (junction (at 104.14 138.43) (diameter 0) (color 0 0 0 0)
-  )
-  (junction (at 104.14 133.35) (diameter 0) (color 0 0 0 0)
-  )
-  (junction (at 134.62 125.73) (diameter 0) (color 0 0 0 0)
-  )
-  (junction (at 78.74 123.19) (diameter 0) (color 0 0 0 0)
   )
   (junction (at 113.03 115.57) (diameter 0) (color 0 0 0 0)
@@
     )
   )
-  (symbol (lib_id "Simulation_SPICE:PNP") (at 111.76 138.43 0) (mirror x) (unit 1)
-    (in_bom yes) (on_board yes) (dnp no)
-    (property "Reference" "Q2" (at 110.49 134.62 0)
-      (effects (font (size 1.27 1.27)) (justify left))
-    )
-    (property "Value" "PNP" (at 116.84 137.16 0)
-      (effects (font (size 1.27 1.27)) (justify left) hide)
-    )
-    (property "Footprint" "" (at 147.32 138.43 0)
-      (effects (font (size 1.27 1.27)) hide)
-    )
-    (property "Datasheet" "~" (at 147.32 138.43 0)
-      (effects (font (size 1.27 1.27)) hide)
-    )
-    (property "Sim.Device" "PNP" (at 111.76 138.43 0)
-      (effects (font (size 1.27 1.27)) hide)
-    )
-    (property "Sim.Type" "GUMMELPOON" (at 111.76 138.43 0)
-      (effects (font (size 1.27 1.27)) hide)
-    )
-    (property "Sim.Pins" "1=C 2=B 3=E" (at 111.76 138.43 0)
-      (effects (font (size 1.27 1.27)) hide)
-    )
-    (pin "2")
-    (pin "1")
-    (pin "3")
-    (instances
-      (project "NixiePowerSupply"
-        (path "/51ff178e-c901-4ddf-a818-5beaa90f4a97"
-          (reference "Q2") (unit 1)
-        )
-      )
-    )
-  )
   (symbol (lib_id "Device:R") (at 129.54 147.32 0) (unit 1)
     (in_bom yes) (on_board yes) (dnp no)
@@
       (effects (font (size 1.27 1.27)) (justify left) hide)
     )
-    (property "Footprint" "" (at 113.9952 123.19 0)
+    (property "Footprint" "Capacitor_THT:CP_Radial_D6.3mm_P2.50mm" (at 113.9952 123.19 0)
       (effects (font (size 1.27 1.27)) hide)
     )
@@
     )
   )
+  (symbol (lib_id "Transistor_BJT:2N3905") (at 111.76 138.43 0) (mirror x) (unit 1)
+    (in_bom yes) (on_board yes) (dnp no)
+    (property "Reference" "Q2" (at 110.49 134.62 0)
+      (effects (font (size 1.27 1.27)) (justify left))
+    )
+    (property "Value" "2N3905" (at 116.84 137.16 0)
+      (effects (font (size 1.27 1.27)) (justify left) hide)
+    )
+    (property "Footprint" "Package_TO_SOT_THT:TO-92_Inline" (at 116.84 136.525 0)
+      (effects (font (size 1.27 1.27) italic) (justify left) hide)
+    )
+    (property "Datasheet" "https://www.nteinc.com/specs/original/2N3905_06.pdf" (at 111.76 138.43 0)
+      (effects (font (size 1.27 1.27)) (justify left) hide)
+    )
+    (pin "2")
+    (pin "3")
+    (pin "1")
+    (instances
+      (project "NixiePowerSupply"
+        (path "/51ff178e-c901-4ddf-a818-5beaa90f4a97"
+          (reference "Q2") (unit 1)
+        )
+      )
+    )
+  )
   (symbol (lib_id "power:GND") (at 121.92 138.43 0) (unit 1)
     (in_bom yes) (on_board yes) (dnp no) (fields_autoplaced)
@@
       (effects (font (size 1.27 1.27)) hide)
     )
-    (property "Footprint" "" (at 125.73 125.73 0)
+    (property "Footprint" "Diode_THT:D_DO-41_SOD81_P7.62mm_Horizontal" (at 125.73 125.73 0)
       (effects (font (size 1.27 1.27)) hide)
     )
@@
       (effects (font (size 1.27 1.27)) hide)
     )
-    (property "Footprint" "" (at 107.95 133.35 0)
+    (property "Footprint" "Diode_THT:D_DO-35_SOD27_P7.62mm_Horizontal" (at 107.95 133.35 0)
       (effects (font (size 1.27 1.27)) hide)
     )
@@
       (effects (font (size 1.27 1.27)) (justify left) hide)
     )
-    (property "Footprint" "" (at 135.5852 133.35 0)
+    (property "Footprint" "Capacitor_THT:CP_Radial_D6.3mm_P2.50mm" (at 135.5852 133.35 0)
       (effects (font (size 1.27 1.27)) hide)
     )
@@
       (effects (font (size 1.27 1.27)) (justify left) hide)
     )
-    (property "Footprint" "" (at 121.92 119.38 0)
-      (effects (font (size 1.27 1.27)) hide)
-    )
+    (property "Footprint" "Inductor_SMD:L_12x12mm_H8mm" (at 121.92 119.38 0)
+      (effects (font (size 1.27 1.27)) hide)
+    )
