File: NixiePowerSupply.kicad_sch (KiCad schematic)
At the start: 16 parts, among them J1 Conn_01x02, J2 Conn_01x02, Q1 IRF740, Q2 2N3905, U1 MC34063AP

Commit message: add ibom
Parts:
- C1: value C_Polarized -> 220uF 16V LESR Polar 6.3x2.5; Link (none) -> https://www.chipdip.ru/product0/9000565757
- C2: value C -> 2200pF, 0805
- C3: value C -> 0.01uF, 0805
- C4: value C_Polarized -> 2.2uF 250V Polar 6.3x2.5; Link (none) -> https://www.chipdip.ru/product0/9000565820
- D1: value D -> UF4004 UF4007, DO-41
- D2: value D -> 1N4148 1N914, DO-35
- J1, J2: value Conn_01x02 -> DG301-5.0-2P
- L1: value L -> 220uH, 12x12
- Q1: value IRF740 -> IRF740, TO-220
- Q2: value 2N3905 -> MPSA55, TO-92
- R1: value R -> 0.33, 0805
- R2: value R -> 1K, 0805
- R3: value R -> 475K, 1%
- R4: value R -> 3K32, 1%
- U1: value MC34063AP -> MC34063
Changed lines of the file:
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@@
       (effects (font (size 1.27 1.27)) (justify left))
     )
-    (property "Value" "C" (at 127 148.59 0)
+    (property "Value" "0.01uF, 0805" (at 127 148.59 0)
       (effects (font (size 1.27 1.27)) (justify left) hide)
     )
@@
       (effects (font (size 1.27 1.27)) (justify left))
     )
-    (property "Value" "Conn_01x02" (at 147.32 128.27 0)
+    (property "Value" "DG301-5.0-2P" (at 147.32 128.27 0)
       (effects (font (size 1.27 1.27)) (justify left) hide)
     )
@@
       (effects (font (size 1.27 1.27)) (justify left))
     )
-    (property "Value" "Conn_01x02" (at 68.58 125.73 0)
+    (property "Value" "DG301-5.0-2P" (at 68.58 125.73 0)
       (effects (font (size 1.27 1.27)) (justify left) hide)
     )
@@
       (effects (font (size 1.27 1.27)) (justify left))
     )
-    (property "Value" "R" (at 132.08 148.59 0)
+    (property "Value" "3K32, 1%" (at 132.08 148.59 0)
       (effects (font (size 1.27 1.27)) (justify left) hide)
     )
@@
       (effects (font (size 1.27 1.27)) (justify left))
     )
-    (property "Value" "C" (at 82.55 138.43 0)
+    (property "Value" "2200pF, 0805" (at 82.55 138.43 0)
       (effects (font (size 1.27 1.27)) (justify left) hide)
     )
@@
       (effects (font (size 1.27 1.27)) (justify left))
     )
-    (property "Value" "C_Polarized" (at 116.84 119.761 0)
+    (property "Value" "220uF 16V LESR Polar 6.3x2.5" (at 116.84 119.761 0)
       (effects (font (size 1.27 1.27)) (justify left) hide)
     )
@@
       (effects (font (size 1.27 1.27)) hide)
     )
+    (property "Link" "https://www.chipdip.ru/product0/9000565757" (at 113.03 119.38 0)
+      (effects (font (size 1.27 1.27)) hide)
+    )
     (pin "1")
     (pin "2")
@@
       (effects (font (size 1.27 1.27)) (justify left))
     )
-    (property "Value" "IRF740" (at 125.73 134.62 0)
+    (property "Value" "IRF740, TO-220" (at 125.73 134.62 0)
       (effects (font (size 1.27 1.27)) (justify left) hide)
     )
@@
       (effects (font (size 1.27 1.27)) (justify left))
     )
-    (property "Value" "R" (at 106.68 143.51 0)
+    (property "Value" "1K, 0805" (at 106.68 143.51 0)
       (effects (font (size 1.27 1.27)) (justify left) hide)
     )
@@
       (effects (font (size 1.27 1.27)) (justify left))
     )
-    (property "Value" "2N3905" (at 116.84 137.16 0)
+    (property "Value" "MPSA55, TO-92" (at 116.84 137.16 0)
       (effects (font (size 1.27 1.27)) (justify left) hide)
     )
@@
       (effects (font (size 1.27 1.27)))
     )
-    (property "Value" "D" (at 125.73 121.92 0)
+    (property "Value" "UF4004 UF4007, DO-41" (at 125.73 121.92 0)
       (effects (font (size 1.27 1.27)) hide)
     )
@@
       (effects (font (size 1.27 1.27)))
     )
-    (property "Value" "R" (at 91.44 111.76 90)
+    (property "Value" "0.33, 0805" (at 91.44 111.76 90)
       (effects (font (size 1.27 1.27)) hide)
     )
@@
       (effects (font (size 1.27 1.27)))
     )
-    (property "Value" "D" (at 107.95 129.54 0)
+    (property "Value" "1N4148 1N914, DO-35" (at 107.95 129.54 0)
       (effects (font (size 1.27 1.27)) hide)
     )
@@
       (effects (font (size 1.27 1.27)) (justify left))
     )
-    (property "Value" "R" (at 132.08 140.97 0)
+    (property "Value" "475K, 1%" (at 132.08 140.97 0)
       (effects (font (size 1.27 1.27)) (justify left) hide)
     )
@@
       (effects (font (size 1.27 1.27)) (justify left))
     )
-    (property "Value" "C_Polarized" (at 138.43 129.921 0)
+    (property "Value" "2.2uF 250V Polar 6.3x2.5" (at 138.43 129.921 0)
       (effects (font (size 1.27 1.27)) (justify left) hide)
     )
@@
       (effects (font (size 1.27 1.27)) hide)
     )
+    (property "Link" "https://www.chipdip.ru/product0/9000565820" (at 134.62 129.54 0)
+      (effects (font (size 1.27 1.27)) hide)
+    )
     (pin "2")
     (pin "1")
@@
       (effects (font (size 1.27 1.27)) (justify left))
     )
-    (property "Value" "L" (at 123.19 120.65 0)
+    (property "Value" "220uH, 12x12" (at 123.19 120.65 0)
       (effects (font (size 1.27 1.27)) (justify left) hide)
     )
@@
       (effects (font (size 1.27 1.27)))
     )
-    (property "Value" "MC34063AP" (at 91.44 130.81 0)
+    (property "Value" "MC34063" (at 91.44 130.81 0)
       (effects (font (size 1.27 1.27)))
     )

Commit message: fix R3, R4
Parts:
- R3: value 475K, 1% -> 470K, 1%
- R4: value 3K32, 1% -> 3K, 1%
Changed lines of the file:
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@@
       (effects (font (size 1.27 1.27)) (justify left))
     )
-    (property "Value" "3K32, 1%" (at 132.08 148.59 0)
+    (property "Value" "3K, 1%" (at 132.08 148.59 0)
       (effects (font (size 1.27 1.27)) (justify left) hide)
     )
@@
       (effects (font (size 1.27 1.27)) (justify left))
     )
-    (property "Value" "475K, 1%" (at 132.08 140.97 0)
-      (effects (font (size 1.27 1.27)) (justify left) hide)
-    )
+    (property "Value" "470K, 1%" (at 132.08 140.97 0)
+      (effects (font (size 1.27 1.27)) (justify left) hide)
+    )

Commit message: fix links in bom
Parts:
- C2: Link (none) -> https://www.chipdip.ru/product/grm2165c1h222j
- C3: Link (none) -> https://www.chipdip.ru/product/grm2195c1h103j
- D1: Link (none) -> https://aliexpress.ru/item/4000798077881.html?spm=a2g2w.ord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
- L1: Link (none) -> https://aliexpress.ru/item/1005001699203887.html?spm=a2g2w.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
- Q1: Link (none) -> https://www.platan.ru/cgi-bin/qwery.pl/id=318826868
- Q2: value MPSA55, TO-92 -> MPSA56, TO-92; Link (none) -> https://www.chipdip.ru/product/mpsa56-diotec
- R1: Link (none) -> https://aliexpress.ru/item/1005001794062302.html?spm=a2g2w.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
- R3, R4: Link (none) -> https://aliexpress.ru/item/32847096736.html?spm=a2g2w.order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
Changed lines of the file:
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@@
+      (effects (font (size 1.27 1.27)) hide)
+    )
+    (property "Link" "https://www.chipdip.ru/product/grm2195c1h103j" (at 123.19 147.32 0)
       (effects (font (size 1.27 1.27)) hide)
     )
@@
       (effects (font (size 1.27 1.27)) hide)
     )
+    (property "Link" "https://aliexpress.ru/item/32847096736.html?spm=a2g2w.orderdetail.0.0.961e4aa6zXOBsP&sku_id=65227930969" (at 129.54 147.32 0)
+      (effects (font (size 1.27 1.27)) hide)
+    )
     (pin "1")
     (pin "2")
@@
     )
     (property "Datasheet" "~" (at 78.74 137.16 0)
+      (effects (font (size 1.27 1.27)) hide)
+    )
+    (property "Link" "https://www.chipdip.ru/product/grm2165c1h222j" (at 78.74 137.16 0)
       (effects (font (size 1.27 1.27)) hide)
     )
@@
       (effects (font (size 1.27 1.27)) (justify left) hide)
     )
+    (property "Link" "https://www.platan.ru/cgi-bin/qwery.pl/id=318826868" (at 119.38 133.35 0)
+      (effects (font (size 1.27 1.27)) hide)
+    )
     (pin "1")
     (pin "3")
@@
       (effects (font (size 1.27 1.27)) (justify left))
     )
-    (property "Value" "MPSA55, TO-92" (at 116.84 137.16 0)
+    (property "Value" "MPSA56, TO-92" (at 116.84 137.16 0)
       (effects (font (size 1.27 1.27)) (justify left) hide)
     )
@@
       (effects (font (size 1.27 1.27)) (justify left) hide)
     )
+    (property "Link" "https://www.chipdip.ru/product/mpsa56-diotec" (at 111.76 138.43 0)
+      (effects (font (size 1.27 1.27)) hide)
+    )
     (pin "2")
     (pin "3")
@@
       (effects (font (size 1.27 1.27)) hide)
     )
+    (property "Link" "https://aliexpress.ru/item/4000798077881.html?spm=a2g2w.orderdetail.0.0.635f4aa6UDS5z0&sku_id=10000008048731253" (at 125.73 125.73 0)
+      (effects (font (size 1.27 1.27)) hide)
+    )
     (pin "1")
     (pin "2")
@@
       (effects (font (size 1.27 1.27)) hide)
     )
+    (property "Link" "https://aliexpress.ru/item/1005001794062302.html?spm=a2g2w.orderdetail.0.0.3b194aa6BKKUxl&sku_id=12000017594821115" (at 91.44 115.57 90)
+      (effects (font (size 1.27 1.27)) hide)
+    )
     (pin "2")
     (pin "1")
@@
       (effects (font (size 1.27 1.27)) hide)
     )
+    (property "Link" "https://aliexpress.ru/item/32847096736.html?spm=a2g2w.orderdetail.0.0.961e4aa6m8WYZn&sku_id=12000030032474500" (at 129.54 139.7 0)
+      (effects (font (size 1.27 1.27)) hide)
+    )
     (pin "2")
     (pin "1")
@@
       (effects (font (size 1.27 1.27)) hide)
     )
+    (property "Link" "https://aliexpress.ru/item/1005001699203887.html?spm=a2g2w.orderdetail.0.0.1cbb4aa6UPdjMI&sku_id=12000017203437476" (at 121.92 119.38 0)
+      (effects (font (size 1.27 1.27)) hide)
+    )
